Commit message: [REF] Remove unused ros2_control node and associated joint definitions from launch and URDF files

File: ros2_ws/src/dls_resources_piper_description/urdf/piper_description.xacro (robot description, xacro)
@@ -537,67 +537,3 @@
     <xacro:transmission_block tran_name="tran7" joint_name="joint7" motor_name="motor7" />
   </xacro:if>
-  <ros2_control name="MockSystem" type="system">
-    <hardware>
-      <plugin>mock_components/GenericSystem</plugin>
-    </hardware>
-    <joint name="joint1">
-      <command_interface name="position" />
-      <state_interface name="position">
-        <param name="initial_value">0.0</param>
-      </state_interface>
-      <state_interface name="velocity" />
-    </joint>
-    <joint name="joint2">
-      <command_interface name="position" />
-      <state_interface name="position">
-        <param name="initial_value">0.0</param>
-      </state_interface>
-      <state_interface name="velocity" />
-    </joint>
-    <joint name="joint3">
-      <command_interface name="position" />
-      <state_interface name="position">
-        <param name="initial_value">0.0</param>
-      </state_interface>
-      <state_interface name="velocity" />
-    </joint>
-    <joint name="joint4">
-      <command_interface name="position" />
-      <state_interface name="position">
-        <param name="initial_value">0.0</param>
-      </state_interface>
-      <state_interface name="velocity" />
-    </joint>
-    <joint name="joint5">
-      <command_interface name="position" />
-      <state_interface name="position">
-        <param name="initial_value">0.0</param>
-      </state_interface>
-      <state_interface name="velocity" />
-    </joint>
-    <joint name="joint6">
-      <command_interface name="position" />
-      <state_interface name="position">
-        <param name="initial_value">0.0</param>
-      </state_interface>
-      <state_interface name="velocity" />
-    </joint>
-    <xacro:if value="$(arg gripper)">
-      <joint name="joint7">
-        <command_interface name="position" />
-        <state_interface name="position">
-          <param name="initial_value">0.0</param>
-        </state_interface>
-        <state_interface name="velocity" />
-      </joint>
-      <joint name="joint8">
-        <param name="mimic">joint7</param>
-        <param name="multiplier">-1.0</param>
-        <state_interface name="position">
-          <param name="initial_value">0.0</param>
-        </state_interface>
-        <state_interface name="velocity" />
-      </joint>
-    </xacro:if>
-  </ros2_control>
 </robot>
